Commit message: ignition bridge for thruster rpm

File: hippo_sim/models/thruster/urdf/thruster_macro.xacro (robot description, xacro)
@@ -97,18 +97,16 @@
         <gazebo>
             <plugin filename="thruster" name="hippo_gz_plugins::thruster">
-                <thruster_config>
-                    <link>${propeller_link}</link>
-                    <joint>${propeller_joint}</joint>
-                    <linear_coeff>${thrust_linear_coeff}</linear_coeff>
-                    <quadratic_coeff>${thrust_quadratic_coeff}</quadratic_coeff>
-                    <torque_coeff>${torque_constant}</torque_coeff>
-                    <rpm_scaler>${rpm_scaler}</rpm_scaler>
-                    <max_rpm>${max_rpm}</max_rpm>
-                    <thruster_number>${number}</thruster_number>
-                    <turning_direction>${turning_direction}</turning_direction>
-                    <propeller_direction>${propeller_direction}</propeller_direction>
-                    <timeconstant_up>${timeconstant_up}</timeconstant_up>
-                    <timeconstant_down>${timeconstant_down}</timeconstant_down>
-                </thruster_config>
+                <link>${propeller_link}</link>
+                <joint>${propeller_joint}</joint>
+                <linear_coeff>${thrust_linear_coeff}</linear_coeff>
+                <quadratic_coeff>${thrust_quadratic_coeff}</quadratic_coeff>
+                <torque_coeff>${torque_constant}</torque_coeff>
+                <rpm_scaler>${rpm_scaler}</rpm_scaler>
+                <max_rpm>${max_rpm}</max_rpm>
+                <thruster_number>${number}</thruster_number>
+                <turning_direction>${turning_direction}</turning_direction>
+                <propeller_direction>${propeller_direction}</propeller_direction>
+                <timeconstant_up>${timeconstant_up}</timeconstant_up>
+                <timeconstant_down>${timeconstant_down}</timeconstant_down>
             </plugin>
         </gazebo>

Commit message: fixed thruster params and adapted mixer matrix.
Scale the inputs depending in number of participating motors in that
degree of freedom.

File: hippo_sim/models/thruster/urdf/thruster_macro.xacro (robot description, xacro)
@@ -99,12 +99,16 @@
                 <link>${propeller_link}</link>
                 <joint>${propeller_joint}</joint>
-                <linear_coeff>${thrust_linear_coeff}</linear_coeff>
-                <quadratic_coeff>${thrust_quadratic_coeff}</quadratic_coeff>
-                <torque_coeff>${torque_constant}</torque_coeff>
-                <rpm_scaler>${rpm_scaler}</rpm_scaler>
-                <max_rpm>${max_rpm}</max_rpm>
+                <publish_rate>50.0</publish_rate>
+                <throttle_cmd_base_topic>throttle_cmd</throttle_cmd_base_topic>
+                <rpm_base_topic>rpm</rpm_base_topic>
+                <thrust_base_topic>thrust</thrust_base_topic>
                 <thruster_number>${number}</thruster_number>
                 <turning_direction>${turning_direction}</turning_direction>
                 <propeller_direction>${propeller_direction}</propeller_direction>
+                <maximum_rpm>${max_rpm}</maximum_rpm>
+                <rpm_scaler>${rpm_scaler}</rpm_scaler>
+                <torque_coeff>${torque_constant}</torque_coeff>
+                <linear_coeff>${thrust_linear_coeff}</linear_coeff>
+                <quadratic_coeff>${thrust_quadratic_coeff}</quadratic_coeff>
                 <timeconstant_up>${timeconstant_up}</timeconstant_up>
                 <timeconstant_down>${timeconstant_down}</timeconstant_down>

File: hippo_sim/models/thruster/urdf/thruster_params.xacro (robot description, xacro)
@@ -5,8 +5,8 @@
     <xacro:property name="thruster_iyy" value="1e-6" />
     <xacro:property name="thruster_izz" value="1e-6" />
-    <xacro:property name="thrust_linear_coeff" value="2.6e-5" />
-    <xacro:property name="thrust_quadratic_coeff" value="4.2e-3" />
+    <xacro:property name="thrust_linear_coeff" value="4.2e-1" />
+    <xacro:property name="thrust_quadratic_coeff" value="2.6e-4" />
     <xacro:property name="torque_constant" value="1e-2" />
-    <xacro:property name="rpm_scaler" value="1" />
+    <xacro:property name="rpm_scaler" value="100" />
     <xacro:property name="max_rpm" value="3000" />
     <xacro:property name="timeconstant_up" value="0.05" />

Commit message: more debug messages

File: hippo_sim/models/thruster/urdf/thruster_macro.xacro (robot description, xacro)
@@ -110,4 +110,5 @@
                 <torque_coeff>${torque_constant}</torque_coeff>
                 <linear_coeff>${thrust_linear_coeff}</linear_coeff>
+                <constant_coeff>${thrust_constant_coeff}</constant_coeff>
                 <quadratic_coeff>${thrust_quadratic_coeff}</quadratic_coeff>
                 <timeconstant_up>${timeconstant_up}</timeconstant_up>

File: hippo_sim/models/thruster/urdf/thruster_params.xacro (robot description, xacro)
@@ -5,6 +5,7 @@
     <xacro:property name="thruster_iyy" value="1e-6" />
     <xacro:property name="thruster_izz" value="1e-6" />
-    <xacro:property name="thrust_quadratic_coeff" value="2.6e-3" />
-    <xacro:property name="thrust_linear_coeff" value="4.2e-2" />
+    <xacro:property name="thrust_quadratic_coeff" value="3.313e-3" />
+    <xacro:property name="thrust_linear_coeff" value="0.1086" />
+    <xacro:property name="thrust_constant_coeff" value="-0.8576" />
     <xacro:property name="torque_constant" value="1e-2" />
     <xacro:property name="rpm_scaler" value="1" />
