Commit message: thrusters params from data sheet

File: hippo_sim/models/thruster/urdf/t200_params.xacro (robot description, xacro)
@@ -5,10 +5,16 @@
     <xacro:property name="thruster_iyy" value="1e-6" />
     <xacro:property name="thruster_izz" value="1e-6" />
-    <xacro:property name="thrust_quadratic_coeff" value="3.313e-3" />
-    <xacro:property name="thrust_linear_coeff" value="0.1086" />
-    <xacro:property name="thrust_constant_coeff" value="-0.8576" />
-    <xacro:property name="torque_constant" value="1e-2" />
+    <!-- based on 14V performance data and forced interception at 0.0 -->
+    <xacro:property name="thrust_quadratic_coeff" value="0.015547" />
+    <xacro:property name="thrust_linear_coeff" value="-0.04243" />
+    <xacro:property name="thrust_constant_coeff" value="0.0" />
+    <xacro:property name="torque_constant" value="0.0" />
+    <!-- for reversed direction:  0.01268 -0.05067 0.0 -->
+    <!-- Throttle = f(revs/s) -->
+    <xacro:property name="velocity_quadratic_coeff" value="1.2679e-4"/>
+    <xacro:property name="velocity_linear_coeff" value="1.1105e-2"/>
+    <xacro:property name="velocity_constant_coeff" value="0.0"/>
     <xacro:property name="rpm_scaler" value="10" />
-    <xacro:property name="max_rpm" value="3000" />
+    <xacro:property name="max_rpm" value="3240" />
     <xacro:property name="timeconstant_up" value="0.00" />
     <xacro:property name="timeconstant_down" value="0.00" />
