Commit message: thrust function is now a function of rotations per second instead of rotational velocity

File: hippo_sim/models/thruster/urdf/thruster_params.xacro (robot description, xacro)
@@ -5,9 +5,9 @@
     <xacro:property name="thruster_iyy" value="1e-6" />
     <xacro:property name="thruster_izz" value="1e-6" />
-    <xacro:property name="thrust_linear_coeff" value="15.89e-5" />
-    <xacro:property name="thrust_quadratic_coeff" value="23.2e-5" />
+    <xacro:property name="thrust_linear_coeff" value="2.6e-5" />
+    <xacro:property name="thrust_quadratic_coeff" value="4.2e-3" />
     <xacro:property name="torque_constant" value="1e-2" />
     <xacro:property name="rpm_scaler" value="1" />
-    <xacro:property name="max_rpm" value="800" />
+    <xacro:property name="max_rpm" value="3000" />
     <xacro:property name="timeconstant_up" value="0.05" />
     <xacro:property name="timeconstant_down" value="0.05" />

Commit message: made mixer thrust function parametrical

File: hippo_sim/models/thruster/urdf/thruster_params.xacro (robot description, xacro)
@@ -5,8 +5,8 @@
     <xacro:property name="thruster_iyy" value="1e-6" />
     <xacro:property name="thruster_izz" value="1e-6" />
-    <xacro:property name="thrust_linear_coeff" value="4.2e-1" />
-    <xacro:property name="thrust_quadratic_coeff" value="2.6e-4" />
+    <xacro:property name="thrust_quadratic_coeff" value="2.6e-3" />
+    <xacro:property name="thrust_linear_coeff" value="4.2e-2" />
     <xacro:property name="torque_constant" value="1e-2" />
-    <xacro:property name="rpm_scaler" value="100" />
+    <xacro:property name="rpm_scaler" value="1" />
     <xacro:property name="max_rpm" value="3000" />
     <xacro:property name="timeconstant_up" value="0.05" />

Commit message: set default thruster timeconstant to zero

File: hippo_sim/models/thruster/urdf/thruster_params.xacro (robot description, xacro)
@@ -10,5 +10,5 @@
     <xacro:property name="rpm_scaler" value="1" />
     <xacro:property name="max_rpm" value="3000" />
-    <xacro:property name="timeconstant_up" value="0.05" />
-    <xacro:property name="timeconstant_down" value="0.05" />
+    <xacro:property name="timeconstant_up" value="0.00" />
+    <xacro:property name="timeconstant_down" value="0.00" />
 </robot>

Commit message: thruster params update

File: hippo_sim/models/thruster/urdf/thruster_params.xacro (robot description, xacro)
@@ -8,4 +8,8 @@
     <xacro:property name="thrust_linear_coeff" value="0.1086" />
     <xacro:property name="thrust_constant_coeff" value="-0.8576" />
+    <!-- Throttle = f(revs/s) -->
+    <xacro:property name="velocity_quadratic_coeff" value="1.2679e-4"/>
+    <xacro:property name="velocity_linear_coeff" value="1.1105e-2"/>
+    <xacro:property name="velocity_constant_coeff" value="0.0"/>
     <xacro:property name="torque_constant" value="1e-2" />
     <xacro:property name="rpm_scaler" value="1" />
