Commit message: update mass to actual value

File: hippo_sim/models/hippo3/urdf/hippo3_params.xacro (robot description, xacro)
@@ -1,5 +1,5 @@
 <?xml version="1.0"?>
 <robot xmlns:xacro="http://www.ros.org/wiki/xacro">
-    <xacro:property name="base_mass" value="1.47" />
+    <xacro:property name="base_mass" value="2.31" />
     <xacro:property name="ixx" value="0.0024" />
     <xacro:property name="iyy" value="0.010717" />
