Commit message: updated world and hippo model

File: hippo_sim/models/hippo3/urdf/hippo3.xacro (robot description, xacro)
@@ -113,5 +113,5 @@
             <buoyancy>
                 <link_name>base_link</link_name>
-                <origin>0 0 0.000</origin>
+                <origin>0 0 0.01</origin>
                 <force_added>0</force_added>
                 <compensation>1.01</compensation>

Commit message: bluerov added

File: hippo_sim/models/hippo3/urdf/hippo3.xacro (robot description, xacro)
@@ -100,8 +100,8 @@
         </visual>
     </gazebo>
-    <xacro:thruster parent="base_link" suffix="port_top" xyz="0 ${thruster_r / 2**0.5} ${thruster_r / 2**0.5}" axis="1 0 0" turning_direction="ccw" propeller_direction="ccw" color="red" number="0" />
-    <xacro:thruster parent="base_link" suffix="starboard_top" xyz="0 -${thruster_r / 2**0.5} ${thruster_r / 2**0.5}" axis="1 0 0" turning_direction="ccw" propeller_direction="cw" color="green" number="1" />
-    <xacro:thruster parent="base_link" suffix="starboard_bot" xyz="0 -${thruster_r / 2**0.5} -${thruster_r / 2**0.5}" axis="1 0 0" turning_direction="ccw" propeller_direction="ccw" color="grey" number="2" />
-    <xacro:thruster parent="base_link" suffix="port_bot" xyz="0 ${thruster_r / 2**0.5} -${thruster_r / 2**0.5}" axis="1 0 0" turning_direction="cw" propeller_direction="ccw" color="grey" number="3" />
+    <xacro:thruster parent="base_link" suffix="port_top" xyz="0 ${thruster_r / 2**0.5} ${thruster_r / 2**0.5}" rpy="0 0 0" turning_direction="ccw" propeller_direction="ccw" color="red" number="0" />
+    <xacro:thruster parent="base_link" suffix="starboard_top" xyz="0 -${thruster_r / 2**0.5} ${thruster_r / 2**0.5}" rpy="0 0 0" turning_direction="ccw" propeller_direction="cw" color="green" number="1" />
+    <xacro:thruster parent="base_link" suffix="starboard_bot" xyz="0 -${thruster_r / 2**0.5} -${thruster_r / 2**0.5}" rpy="0 0 0" turning_direction="ccw" propeller_direction="ccw" color="grey" number="2" />
+    <xacro:thruster parent="base_link" suffix="port_bot" xyz="0 ${thruster_r / 2**0.5} -${thruster_r / 2**0.5}" rpy="0 0 0" turning_direction="cw" propeller_direction="ccw" color="grey" number="3" />
     <xacro:mount parent="base_link" suffix="port_top" xyz="0 ${thruster_r / 2**0.5} ${thruster_r / 2**0.5}" rpy="${radians(-45)} 0 0" />
     <xacro:mount parent="base_link" suffix="starboard_top" xyz="0 -${thruster_r / 2**0.5} ${thruster_r / 2**0.5}" rpy="${radians(45)} 0 0" />

File: hippo_sim/models/thruster/urdf/t200_params.xacro (robot description, xacro)
@@ -9,8 +9,8 @@
     <xacro:property name="thrust_constant_coeff" value="-0.8576" />
     <xacro:property name="torque_constant" value="1e-2" />
-    <xacro:property name="rpm_scaler" value="1" />
+    <xacro:property name="rpm_scaler" value="10" />
     <xacro:property name="max_rpm" value="3000" />
     <xacro:property name="timeconstant_up" value="0.00" />
     <xacro:property name="timeconstant_down" value="0.00" />
-    <xacro:property name="propeller_mesh" value="$(find hippo_sim)/models/thruster/meshes/propeller.dae" />
+    <xacro:property name="propeller_mesh" value="$(find hippo_sim)/models/thruster/meshes/t200_propeller.dae" />
 </robot>

File: hippo_sim/models/thruster/urdf/thruster_macro.xacro (robot description, xacro)
@@ -1,6 +1,5 @@
 <?xml version="1.0"?>
 <robot xmlns:xacro="http://www.ros.org/wiki/xacro">
-    <xacro:macro name="thruster" params="suffix parent xyz axis turning_direction propeller_direction color number">
-        <xacro:include filename="$(find hippo_sim)/models/thruster/urdf/thruster_params.xacro" />
+    <xacro:macro name="thruster" params="model:='generic' suffix parent xyz rpy turning_direction propeller_direction color number">
         <xacro:property name="mount_link" value="${suffix}_thruster_mount_link" />
         <xacro:property name="mount_joint" value="${suffix}_thruster_mount_joint" />
@@ -9,78 +8,84 @@
         <xacro:property name="propeller_link" value="${suffix}_thruster_propeller_link" />
         <xacro:property name="propeller_joint" value="${suffix}_thruster_propeller_joint" />
-        <link name="${mount_link}">
-            <origin xyz="0 0 0" rpy="0 0 0" />
-            <inertial>
-                <mass value="${thruster_mass}" />
-                <inertia ixx="${thruster_ixx}" ixy="0.0" ixz="0.0" iyy="${thruster_iyy}" iyz="0.0" izz="${thruster_izz}" />
-            </inertial>
-            <visual>
-                <geometry>
-                    <mesh filename="$(find hippo_sim)/models/thruster/meshes/motor_mount.dae" />
-                </geometry>
-            </visual>
-        </link>
-        <gazebo reference="${mount_link}">
-            <visual>
-                <material>
-                    <ambient>1 1 1 1</ambient>
-                    <diffuse>1 1 1 1</diffuse>
-                    <specular>1 1 1 1</specular>
-                    <pbr>
-                        <metal>
-                            <metalness>1</metalness>
-                            <roughness>0.5</roughness>
-                            <environment_map>$(find hippo_sim)/models/common/textures/env_map.dds</environment_map>
-                            <albedo_map>$(find hippo_sim)/models/common/textures/grey.png</albedo_map>
-                        </metal>
-                    </pbr>
-                </material>
-            </visual>
-        </gazebo>
-        <joint name="${mount_joint}" type="fixed">
-            <axis xyz="${axis}" />
-            <origin xyz="${xyz}" />
-            <parent link="${parent}" />
-            <child link="${mount_link}" />
-        </joint>
-        <gazebo reference="${mount_joint}">
-            <disableFixedJointLumping>true</disableFixedJointLumping>
-            <preserveFixedJoint>true</preserveFixedJoint>
-        </gazebo>
-        <link name="${hull_link}">
-            <origin xyz="0 0 0" rpy="0 0 0" />
-            <inertial>
-                <mass value="${thruster_mass}" />
-                <inertia ixx="${thruster_ixx}" ixy="0.0" ixz="0.0" iyy="${thruster_iyy}" iyz="0.0" izz="${thruster_izz}" />
-            </inertial>
-            <visual>
-                <geometry>
-                    <mesh filename="$(find hippo_sim)/models/thruster/meshes/motor_hull.dae" />
-                </geometry>
-            </visual>
-        </link>
-        <gazebo reference="${hull_link}">
-            <visual>
-                <material>
-                    <ambient>1 1 1 1</ambient>
-                    <diffuse>1 1 1 1</diffuse>
-                    <specular>1 1 1 1</specular>
-                    <pbr>
-                        <metal>
-                            <metalness>1</metalness>
-                            <roughness>0.5</roughness>
-                            <environment_map>$(find hippo_sim)/models/common/textures/env_map.dds</environment_map>
-                            <albedo_map>$(find hippo_sim)/models/thruster/textures/hippocampus_text.png</albedo_map>
-                        </metal>
-                    </pbr>
-                </material>
-            </visual>
-        </gazebo>
-        <joint name="${hull_joint}" type="continuous">
-            <axis xyz="${axis}" />
-            <origin xyz="${xyz}" />
-            <parent link="${parent}" />
-            <child link="${hull_link}" />
-        </joint>
+        <xacro:if value="${model == 'generic'}">
+            <xacro:include filename="$(find hippo_sim)/models/thruster/urdf/thruster_params.xacro" />
+            <link name="${mount_link}">
+                <origin xyz="0 0 0" rpy="0 0 0" />
+                <inertial>
+                    <mass value="${thruster_mass}" />
+                    <inertia ixx="${thruster_ixx}" ixy="0.0" ixz="0.0" iyy="${thruster_iyy}" iyz="0.0" izz="${thruster_izz}" />
+                </inertial>
+                <visual>
+                    <geometry>
+                        <mesh filename="$(find hippo_sim)/models/thruster/meshes/motor_mount.dae" />
+                    </geometry>
+                </visual>
+            </link>
+            <gazebo reference="${mount_link}">
+                <visual>
+                    <material>
+                        <ambient>1 1 1 1</ambient>
+                        <diffuse>1 1 1 1</diffuse>
+                        <specular>1 1 1 1</specular>
+                        <pbr>
+                            <metal>
+                                <metalness>1</metalness>
+                                <roughness>0.5</roughness>
+                                <environment_map>$(find hippo_sim)/models/common/textures/env_map.dds</environment_map>
+                                <albedo_map>$(find hippo_sim)/models/common/textures/grey.png</albedo_map>
+                            </metal>
+                        </pbr>
+                    </material>
+                </visual>
+            </gazebo>
+            <joint name="${mount_joint}" type="fixed">
+                <axis xyz="1 0 0" />
+                <origin xyz="${xyz}" rpy="${rpy}" />
+                <parent link="${parent}" />
+                <child link="${mount_link}" />
+            </joint>
+            <gazebo reference="${mount_joint}">
+                <disableFixedJointLumping>true</disableFixedJointLumping>
+                <preserveFixedJoint>true</preserveFixedJoint>
+            </gazebo>
+            <link name="${hull_link}">
+                <origin xyz="0 0 0" rpy="0 0 0" />
+                <inertial>
+                    <mass value="${thruster_mass}" />
+                    <inertia ixx="${thruster_ixx}" ixy="0.0" ixz="0.0" iyy="${thruster_iyy}" iyz="0.0" izz="${thruster_izz}" />
+                </inertial>
+                <visual>
+                    <geometry>
+                        <mesh filename="$(find hippo_sim)/models/thruster/meshes/motor_hull.dae" />
+                    </geometry>
+                </visual>
+            </link>
+            <gazebo reference="${hull_link}">
+                <visual>
+                    <material>
+                        <ambient>1 1 1 1</ambient>
+                        <diffuse>1 1 1 1</diffuse>
+                        <specular>1 1 1 1</specular>
+                        <pbr>
+                            <metal>
+                                <metalness>1</metalness>
+                                <roughness>0.5</roughness>
+                                <environment_map>$(find hippo_sim)/models/common/textures/env_map.dds</environment_map>
+                                <albedo_map>$(find hippo_sim)/models/thruster/textures/hippocampus_text.png</albedo_map>
+                            </metal>
+                        </pbr>
+                    </material>
+                </visual>
+            </gazebo>
+            <joint name="${hull_joint}" type="continuous">
+                <axis xyz="1 0 0" />
+                <origin xyz="${xyz}" rpy="${rpy}" />
+                <parent link="${parent}" />
+                <child link="${hull_link}" />
+            </joint>
+        </xacro:if>
+        <xacro:if value="${model == 't200'}">
+            <xacro:include filename="$(find hippo_sim)/models/thruster/urdf/t200_params.xacro" />
+        </xacro:if>
         <link name="${propeller_link}">
             <origin xyz="0 0 0" rpy="0 0 0" />
@@ -91,5 +96,5 @@
             <visual>
                 <geometry>
-                    <mesh filename="$(find hippo_sim)/models/thruster/meshes/propeller_${propeller_direction}.dae" />
+                    <mesh filename="${propeller_mesh}" />
                 </geometry>
             </visual>
@@ -134,6 +139,6 @@
         </gazebo>
         <joint name="${propeller_joint}" type="continuous">
-            <axis xyz="${axis}" />
-            <origin xyz="${xyz}" />
+            <axis xyz="1 0 0" />
+            <origin xyz="${xyz}" rpy="${rpy}" />
             <parent link="${parent}" />
             <child link="${propeller_link}" />
