Commit message: range_sensor framework

File: hippo_sim/models/bluerov/urdf/bluerov.xacro (robot description, xacro)
@@ -66,4 +66,8 @@
             <position>-0.15 0 0</position>
         </plugin>
+        <plugin filename="range_sensor" name="hippo_gz_plugins::range_sensor">
+            <link>base_link</link>
+            <range_topic>range_topic</range_topic>
+        </plugin>
     </gazebo>
 </robot>

Commit message: completed range sensor plugin

File: hippo_sim/models/bluerov/urdf/bluerov.xacro (robot description, xacro)
@@ -69,4 +69,21 @@
             <link>base_link</link>
             <range_topic>range_topic</range_topic>
+            <update_rate>20.0</update_rate>
+            <model name="range_tag_00">
+                <link>base_link</link>
+                <id>0</id>
+            </model>
+            <model name="range_tag_01">
+                <link>base_link</link>
+                <id>1</id>
+            </model>
+            <model name="range_tag_02">
+                <link>base_link</link>
+                <id>2</id>
+            </model>
+            <model name="range_tag_03">
+                <link>base_link</link>
+                <id>3</id>
+            </model>
         </plugin>
     </gazebo>
